File: boards/ZynthianIO/ZynthianIO.kicad_pcb (KiCad board)
At the start: 2 copper layers, 75 x 78 mm, 32 parts, among them J1 Btn-1, J10 Ctrl-2, J11 Display, J2 Raspberry_Pi_2_3, J3 Btn-2, J7 Ctrl-3, J8 Ctrl-4, J9 Ctrl-1, U1 MCP23017_SP, U3 74LS14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

Commit message: Using 74LS07 OC buffer to avoid excessive LED currents
Parts:
- removed U3: 74LS14, Package_DIP:DIP-14_W7.62mm
- added U2: 74LS07, Package_DIP:DIP-14_W7.62mm, F.Cu at (206.2, 105.5)
- MH1, MH2, MH3, MH4: value MountingHole_2.7mm_M2.5 -> MountingHole
- moved C4 5.01 mm to (221.8, 85.2)
Connections:
- MIDI1 pad 4: GND -> unconnected-(MIDI1-Pin_4-Pad4)
- MIDI1 pad 6: GND -> +5V
- MIDI2 pad 4: GND -> unconnected-(MIDI2-Pin_4-Pad4)
- MIDI2 pad 6: GND -> +5V
- MIDI3 pad 4: GND -> unconnected-(MIDI3-Pin_4-Pad4)
- MIDI3 pad 6: GND -> +5V
Routing:
- net +5V: track 126.4 -> 181.8 mm
- net GND: track 17.1 -> 3.81 mm
- net Net-(U3-Pad2): track 2.54 -> 0.00 mm
- net Net-(U3-Pad11): track 2.54 -> 0.00 mm
- net /MIDI_IN: track 53.9 -> 55.0 mm
